File: UCC_50xx_driver_github.kicad_pcb (KiCad board)
At the start: 4 copper layers, 112.6 x 63 mm, 73 parts, among them Q1_Gate1 TestPoint, Q1_Gate2 OUT-, Q1_Gate3 OUT+, Q1_in+1 TestPoint, Q1_in+2 IN+, Q1_in-1 TestPoint, Q1_in-2 IN-, Q3_1 2STF1360, U1_1 MGJ2D051509SC, U1_3 UCC5350MCD, U5 MMSZ3V3T1G

Commit message: Add files via upload
Parts:
- moved Q1_Gate2 48.5 mm to (135.6, 45.8), turned to 0 degrees
- moved Q1_Gate3 38.2 mm to (121.4, 45.8), turned to 180 degrees
- moved TP3 13.8 mm to (153.8, 86.5)
- moved TP1 13.2 mm to (54.1, 85.9)
- moved GND1 12.0 mm to (56.5, 77.9)
- moved GND1_tp1 11.4 mm to (66.1, 78.4)
- moved VAUX1 9.48 mm to (66.1, 69.3)
- moved VAUX1_5V1 9.28 mm to (56.4, 69.4)
- moved Q1_in-2 6.58 mm to (56.3, 60.7)
- moved Q1_in-1 6.38 mm to (66.0, 60.9)
- moved TP4 5.30 mm to (153.9, 44.3)
- moved Q1_in+2 5.10 mm to (56.4, 51.7)
- moved Q1_in+1 3.48 mm to (66.2, 53.3)
Routing:
- net Net-(Q1_Gate3-Pin_1): track 74.5 -> 29.9 mm
- net GND1: track 37.0 -> 24.2 mm, vias 119 -> 86
- net Net-(Q1_in-2-Pin_1): track 40.0 -> 34.7 mm, vias 0 -> 2
- net Net-(Q1_in+2-Pin_1): track 33.3 -> 31.9 mm, vias 0 -> 2
- net GND2: track 53.8 -> 53.7 mm, vias 143 -> 106
- net unconnected-(TP3-Pin_1-Pad1): vias 0 -> 5
- net unconnected-(TP1-Pin_1-Pad1): vias 1 -> 0
- net VAUX: vias 0 -> 7
Other:
- board size 112.6 x 63 mm -> 107.8 x 50.3 mm
